Commit message: add S10 Ultra + M300 cloud merger for GroundGrid ground segmentation

File: omorobot/omorobot_description/urdf/DONKEYBOTI.urdf (robot description, URDF)
Before this commit: robot DONKEYBOTI, 10 links, 9 joints
Links:
- removed link s10_ultra_left_optical
- removed link s10_ultra_link
- removed link s10_ultra_right_optical
Joints:
- removed joint s10_ultra_joint
- removed joint s10_ultra_left_optical_joint
- removed joint s10_ultra_right_optical_joint
